Commit message: Add files via upload

File: my_robot/urdf/my_robot.xacro (robot description, xacro)
@@ -58,4 +58,5 @@
         <box size=".4 .2 .1"/>
       </geometry>
+      <material name="Orange" />
     </visual>
     <collision name='back_caster_collision'>
@@ -105,4 +106,5 @@
         <cylinder radius="0.1" length="0.05" />
       </geometry>
+      <material name="Blue" />
     </visual>
   </link>
@@ -128,4 +130,5 @@
         <cylinder radius="0.1" length="0.05" />
       </geometry>
+      <material name="Blue"/>
     </visual>
   </link>
@@ -151,4 +154,5 @@
 	<box size="0.05 0.05 0.05"/>
       </geometry>
+      <material name="Red"/>
     </visual>
   </link>
@@ -176,3 +180,15 @@
     </visual>
   </link>
+  <gazebo reference="camera">
+    <material>Gazebo/Red</material>
+  </gazebo>
+  <gazebo reference="right_wheel">
+    <material>Gazebo/Blue</material>
+  </gazebo>
+  <gazebo reference="left_wheel">
+    <material>Gazebo/Blue</material>
+  </gazebo>
+  <gazebo reference="chassis">
+    <material>Gazebo/Orange</material>
+  </gazebo>
 </robot>

Commit message: Add files via upload

File: my_robot/urdf/my_robot.xacro (robot description, xacro)
@@ -36,4 +36,9 @@
     <axis xyz="0 1 0" rpy="0 0 0"/>
   </joint>
+  <joint name="camera_optical_joint" type="fixed">
+    <origin xyz="0 0 0" rpy="-1.5707 0 -1.5707"/>
+    <parent link="chassis"/>
+    <child link="camera_link_optical"/>
+  </joint>
   <link name='chassis'>
     <pose>0 0 0.1 0 0 0</pose>
@@ -180,4 +185,6 @@
     </visual>
   </link>
+  <link name="camera_link_optical">
+  </link>
   <gazebo reference="camera">
     <material>Gazebo/Red</material>
